File: PCB/TP_DCI.sch (KiCad schematic (older format))
At the start: 56 parts, among them K1 G5V-2-5DC, K2 G5V-2-5DC, P1 Conn_02x20, P2 Conn_02x20, Q1 BC817W, Q2 BC817W, U1 PS2805-4, U2 ACS725xLCTR-10AU, U4 ACS725xLCTR-10AU, U5 24AA1025, U6 DS3231

Commit message: actualizacion de esquematico con nuevos componentes, se agregan vias termicas en PCB
Parts:
- removed AI2: TB_1X2, Libreria_EDU_CIAA_NXP:bornier2, symbol w_device:TB_1X2
- removed DOB1: 01x06, Connector_PinHeader_2.54mm:PinHeader_2x03_P2.54mm_Vertical, symbol Connector_Generic:Conn_02x03_Odd_Even
- removed K1, K2: G5V-2-5DC, Relay_THT:Relay_DPDT_Omron_G5V-2, symbol g5v-2-ima:G5V-2-IMA
- removed P1, P2: Conn_02x20, Connector_PinHeader_2.54mm:PinHeader_2x20_P2.54mm_Vertical, symbol Connector_Generic:Conn_02x20_Odd_Even
- removed unit 4 of U1
- added AI1-1, AI2+1, AI2-1: TB_1X1, CIAA_footprints:wurth_connector, symbol Connector:Screw_Terminal_01x01
- added F1, F2, F3, F4: Fiducial, Fiducial:Fiducial_0.5mm_Mask1mm, symbol Mechanical:Fiducial
- added H1, H2, H3, H4, H5, H6, H7, H8: MountingHole, MountingHole:MountingHole_2.1mm, symbol Mechanical:MountingHole
- added J8, J9: Molex_KK254, Connector_Molex:Molex_KK-254_AE-6410-04A_1x04_P2.54mm_Vertical, symbol Connector:Conn_01x04_Male
- added K1, K2: G5V-1, Relay_THT:Relay_SPDT_Omron_G5V-1, symbol Relay:G5V-1
- added P1: Conn_Poncho2P_2x_20x2, Poncho_Esqueleto:Conn_Poncho_SinBorde, symbol Poncho_Esqueleto:Conn_Poncho2P_2x_20x2
- AI1+1: renamed from AI1; value TB_1X2 -> TB_1X1; footprint Libreria_EDU_CIAA_NXP:bornier2 -> CIAA_footprints:wurth_connector; symbol w_device:TB_1X2 -> Connector:Screw_Terminal_01x01
- JP1: footprint Jumper:SolderJumper-2_P1.3mm_Open_Pad1.0x1.5mm -> Connector_PinHeader_2.54mm:PinHeader_1x02_P2.54mm_Vertical
- LED1, LED2, LED3: footprint LED_SMD:LED_0603_1608Metric -> LED_SMD:LED_0805_2012Metric
- renumbered DO1A1 to DO1, DO2A1 to DO2
Connections:
- net +3V3: now also R18.1, P1.1 (+3.3V), P1.41 (+3.3V); no longer C4.1, C5.1, R18.2
- net +5V: now also K1.2, K2.2, P1.2 (+5V), P1.42 (+5V)
- net ADC_CH1: now also J9.1 (Pin_1), P1.13 (ADC1); no longer U2.7 (VIOUT)
- net ADC_CH2: now also J9.4 (Pin_4), P1.11 (ADC2); no longer U4.7 (VIOUT)
- net GND: now also P1.28 (GND), P1.30 (GND), P1.32 (GND), P1.4 (GND), P1.43 (GND), P1.45 (GND), P1.47 (GND), P1.77 (GND), P1.79 (GND)
- net GNDA: now also J9.3 (Pin_3), P1.12 (GNDA), P1.14 (GNDA); no longer C1.2, C2.2, C3.2, C6.2, U2.5 (GND), U4.5 (GND)
- net GPIO1: now also P1.72 (GPIO1)
- net GPIO2: now also P1.71 (GPIO2)
- net GPIO3: now also P1.74 (GPIO3)
- net GPIO5: now also P1.76 (GPIO5)
- net GPIO7: now also P1.78 (GPIO7)
- net GPIO8: now also P1.80 (GPIO8)
- net SCL: now also P1.21 (i2cSCL)
- net SDA: now also P1.19 (i2cSDA)
- net VDDA: now also J9.2 (Pin_2), P1.17 (VDDA); no longer C1.1, C2.1, U2.8 (VCC), U4.8 (VCC)
- net at D1.2 (A), D2.1 (K), Q1.3 (C): now also K1.9
- net at U2.3 (IP-), U2.4 (IP-): now also AI1-1.1 (Pin_1); no longer AI1+1.2
- net at U4.1 (IP+), U4.2 (IP+): now also AI2+1.1 (Pin_1)
- net at U4.3 (IP-), U4.4 (IP-): now also AI2-1.1 (Pin_1)
- net at BAT1.1 (+), U6.14 (VBAT): now also JP1.1; no longer JP1.2
- net at D3.2 (A), D4.1 (K), Q2.3 (C): now also K2.9
- net at D5.2 (A): now also R18.2; no longer R18.1
- net at D5.1 (K): now also JP1.2; no longer JP1.1
- net COM1A renamed COM1
- net COM1: now also K1.5, K1.6
- net COM2A renamed COM2
- net COM2: now also K2.5, K2.6
- net NA1A renamed NA1
- net NA1: now also K1.10
- net NA2A renamed NA2
- net NA2: now also K2.10
- net NC1A renamed NC1
- net NC1: now also K1.1
- net NC2A renamed NC2
- net NC2: now also K2.1
- new net: C1.1, C2.1, J8.2 (Pin_2), U2.8 (VCC), U4.8 (VCC)
- new net: C1.2, C2.2, C3.2, C6.2, J8.3 (Pin_3), U2.5 (GND), U4.5 (GND)
- new net +3.3V: C4.1, C5.1
- new net ANALOG_1: J8.1 (Pin_1), U2.7 (VIOUT)
- new net ANALOG_2: J8.4 (Pin_4), U4.7 (VIOUT)
- no-connect marks 50 -> 56
Other:
- note added: "BOTTOM"
- note added: "Cable apantalaldo\npor pares\n"
- note added: "Canales analogicos"
- note added: "Capacitores de\ndesacople Vcc 3,3V"
- note added: "EDU-CIAA : PONCHO FOTOVOLTAICO"
- note added: "Fiduciales\n"
- note added: "Orificios de montaje"
- note added: "PCB EXTERNO"
- note added: "TOP"
- note removed: "Capacitores de desacople ADC"
- note removed: "Capacitores de desacople Vcc 3,3V"
- moved on the sheet: BAT1, C1, C2, C3, C4, C5, C6, D3, D4, D5, DI1, DI2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
